File: Adapter-IO4-35mm.brd (EAGLE design)
At the start: 30.9 x 31.9 mm, 3 parts

Commit message: added values for connectors
Parts:
- J4: value (none) -> RJ45
- JP1: value (none) -> 3.5mm
Changed lines of the file:
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@@
 <elements>
 <element name="U$1" library="SPCoast" package="OSHW-LOGO-M" value="DOC-OSHW-LOGO-M" x="3.81" y="16.51"/>
-<element name="JP1" library="SPCoast" package="SCREWTERMINAL-3.5MM-6" value="" x="7.62" y="3.81"/>
-<element name="J4" library="SPCoast" package="RJ25-PANEL" value="" x="15.24" y="26.67" smashed="yes" rot="R180">
+<element name="JP1" library="SPCoast" package="SCREWTERMINAL-3.5MM-6" value="3.5mm" x="7.62" y="3.81"/>
+<element name="J4" library="SPCoast" package="RJ25-PANEL" value="RJ45" x="15.24" y="26.67" smashed="yes" rot="R180">
 <attribute name="NAME" x="13.335" y="29.21" size="1.778" layer="25"/>
 <attribute name="VALUE" x="22.225" y="34.29" size="1.778" layer="27" rot="R180"/>

Commit message: normalized values
Parts:
- J4: value RJ45 -> RJ12/6
- U$1: value DOC-OSHW-LOGO-M -> OSHW
Changed lines of the file:
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@@
 </autorouter>
 <elements>
-<element name="U$1" library="SPCoast" package="OSHW-LOGO-M" value="DOC-OSHW-LOGO-M" x="3.81" y="16.51"/>
+<element name="U$1" library="SPCoast" package="OSHW-LOGO-M" value="OSHW" x="3.81" y="16.51"/>
 <element name="JP1" library="SPCoast" package="SCREWTERMINAL-3.5MM-6" value="3.5mm" x="7.62" y="3.81"/>
-<element name="J4" library="SPCoast" package="RJ25-PANEL" value="RJ45" x="15.24" y="26.67" smashed="yes" rot="R180">
+<element name="J4" library="SPCoast" package="RJ25-PANEL" value="RJ12/6" x="15.24" y="26.67" smashed="yes" rot="R180">
 <attribute name="NAME" x="13.335" y="29.21" size="1.778" layer="25"/>
 <attribute name="VALUE" x="22.225" y="34.29" size="1.778" layer="27" rot="R180"/>
